File: ErgonomicGamepad.kicad_pcb (KiCad board)
At the start: 2 copper layers, 54 parts, among them J1 USB_C_Receptacle_USB2.0_16P, J2 Conn_01x08, J3 Conn_01x08, J4 Conn_01x08, J5 AVR-ISP-6, J6 Conn_01x08, J7 Conn_01x02, U1 ATmega32U4-A, Y1 Crystal

Commit message: chore: pre-layout baseline (no errors, no warnings, no tech debt)
Parts:
- added JP1: SolderJumper_2_Open, Jumper:SolderJumper-2_P1.3mm_Open_Pad1.0x1.5mm, F.Cu at (120.2, 47.8)
- added SW09: SW_DIP_x01, Switch_Keyboard_Hotswap_Kailh:SW_Hotswap_Kailh_MX_Plated_1.00u, F.Cu at (77.0, 62.3)
- added SW1: SW_DIP_x01, Switch_Keyboard_Hotswap_Kailh:SW_Hotswap_Kailh_MX_Plated_1.00u, F.Cu at (60.4, 46.8)
- added SW10: SW_DIP_x01, Switch_Keyboard_Hotswap_Kailh:SW_Hotswap_Kailh_MX_Plated_1.00u, F.Cu at (77.0, 77.9)
- added SW11: SW_DIP_x01, Switch_Keyboard_Hotswap_Kailh:SW_Hotswap_Kailh_MX_Plated_1.00u, F.Cu at (77.0, 93.4)
- added SW12: SW_DIP_x01, Switch_Keyboard_Hotswap_Kailh:SW_Hotswap_Kailh_MX_Plated_1.00u, F.Cu at (77.0, 109.0)
- added SW13: SW_DIP_x01, Switch_Keyboard_Hotswap_Kailh:SW_Hotswap_Kailh_MX_Plated_1.00u, F.Cu at (77.0, 124.5)
- added SW14: SW_DIP_x01, Switch_Keyboard_Hotswap_Kailh:SW_Hotswap_Kailh_MX_Plated_1.00u, F.Cu at (77.0, 140.1)
- added SW15: SW_DIP_x01, Switch_Keyboard_Hotswap_Kailh:SW_Hotswap_Kailh_MX_Plated_1.00u, F.Cu at (93.6, 46.8)
- added SW16: SW_DIP_x01, Switch_Keyboard_Hotswap_Kailh:SW_Hotswap_Kailh_MX_Plated_1.00u, F.Cu at (93.6, 62.3)
- added SW17: SW_DIP_x01, Switch_Keyboard_Hotswap_Kailh:SW_Hotswap_Kailh_MX_Plated_1.00u, F.Cu at (93.6, 77.9)
- added SW18: SW_DIP_x01, Switch_Keyboard_Hotswap_Kailh:SW_Hotswap_Kailh_MX_Plated_1.00u, F.Cu at (93.6, 93.4)
- added SW19: SW_DIP_x01, Switch_Keyboard_Hotswap_Kailh:SW_Hotswap_Kailh_MX_Plated_1.00u, F.Cu at (93.6, 109.0)
- added SW2: SW_DIP_x01, Switch_Keyboard_Hotswap_Kailh:SW_Hotswap_Kailh_MX_Plated_1.00u, F.Cu at (60.4, 62.3)
- added SW20: SW_DIP_x01, Switch_Keyboard_Hotswap_Kailh:SW_Hotswap_Kailh_MX_Plated_1.00u, F.Cu at (93.6, 124.5)
- added SW21: SW_DIP_x01, Switch_Keyboard_Hotswap_Kailh:SW_Hotswap_Kailh_MX_Plated_1.00u, F.Cu at (93.6, 140.1)
- added SW22: SW_DIP_x01, Switch_Keyboard_Hotswap_Kailh:SW_Hotswap_Kailh_MX_Plated_1.00u, F.Cu at (110.3, 46.8)
- added SW23: SW_DIP_x01, Switch_Keyboard_Hotswap_Kailh:SW_Hotswap_Kailh_MX_Plated_1.00u, F.Cu at (110.3, 62.3)
- added SW24: SW_DIP_x01, Switch_Keyboard_Hotswap_Kailh:SW_Hotswap_Kailh_MX_Plated_1.00u, F.Cu at (110.3, 77.9)
- added SW3: SW_DIP_x01, Switch_Keyboard_Hotswap_Kailh:SW_Hotswap_Kailh_MX_Plated_1.00u, F.Cu at (60.4, 77.9)
- added SW4: SW_DIP_x01, Switch_Keyboard_Hotswap_Kailh:SW_Hotswap_Kailh_MX_Plated_1.00u, F.Cu at (60.4, 93.4)
- added SW5: SW_DIP_x01, Switch_Keyboard_Hotswap_Kailh:SW_Hotswap_Kailh_MX_Plated_1.00u, F.Cu at (60.4, 109.0)
- added SW6: SW_DIP_x01, Switch_Keyboard_Hotswap_Kailh:SW_Hotswap_Kailh_MX_Plated_1.00u, F.Cu at (60.4, 124.5)
- added SW7: SW_DIP_x01, Switch_Keyboard_Hotswap_Kailh:SW_Hotswap_Kailh_MX_Plated_1.00u, F.Cu at (60.4, 140.1)
- added SW8: SW_DIP_x01, Switch_Keyboard_Hotswap_Kailh:SW_Hotswap_Kailh_MX_Plated_1.00u, F.Cu at (77.0, 46.8)
- added SWR1: SW_Push, Button_Switch_SMD:SW_SPST_TL3342, F.Cu at (122.8, 42.5)
- Y1: footprint Crystal:Crystal_SMD_3225-4Pin_3.2x2.5mm -> Crystal:Crystal_SMD_3215-2Pin_3.2x1.5mm
Connections:
- U1 pad 18: unconnected-(U1-PD0-Pad18) -> /COL6
- U1 pad 19: unconnected-(U1-PD1-Pad19) -> /COL5
- U1 pad 20: unconnected-(U1-PD2-Pad20) -> /COL4
- U1 pad 21: unconnected-(U1-PD3-Pad21) -> /COL3
- U1 pad 22: /COL5 -> /COL1
- U1 pad 25: /COL4 -> /COL2
- U1 pad 26: /COL6 -> unconnected-(U1-PD6-Pad26)
- U1 pad 28: /COL1 -> unconnected-(U1-PB4-Pad28)
- U1 pad 29: /COL2 -> unconnected-(U1-PB5-Pad29)
- U1 pad 30: /COL3 -> unconnected-(U1-PB6-Pad30)

Commit message: Snapshot current project state before JLC BOM edits
Parts:
- renumbered SW1 to SW01, SW2 to SW02, SW3 to SW03, SW4 to SW04, SW5 to SW05, SW6 to SW06, SW7 to SW07, SW8 to SW08
Changed lines of the file:
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@@
 		(descr "Kailh keyswitch Hotswap Socket plated holes Keycap 1.00u")
 		(tags "Kailh Keyboard Keyswitch Switch Hotswap Socket Plated Relief Cutout Keycap 1.00u")
-		(property "Reference" "SW7"
+		(property "Reference" "SW07"
 			(at 0 -8 0)
 			(layer "F.SilkS")
@@
 		(descr "Kailh keyswitch Hotswap Socket plated holes Keycap 1.00u")
 		(tags "Kailh Keyboard Keyswitch Switch Hotswap Socket Plated Relief Cutout Keycap 1.00u")
-		(property "Reference" "SW1"
+		(property "Reference" "SW01"
 			(at 0 -8 0)
 			(layer "F.SilkS")
@@
 		(descr "Kailh keyswitch Hotswap Socket plated holes Keycap 1.00u")
 		(tags "Kailh Keyboard Keyswitch Switch Hotswap Socket Plated Relief Cutout Keycap 1.00u")
-		(property "Reference" "SW2"
+		(property "Reference" "SW02"
 			(at 0 -8 0)
 			(layer "F.SilkS")
@@
 		(descr "Kailh keyswitch Hotswap Socket plated holes Keycap 1.00u")
 		(tags "Kailh Keyboard Keyswitch Switch Hotswap Socket Plated Relief Cutout Keycap 1.00u")
-		(property "Reference" "SW6"
+		(property "Reference" "SW06"
 			(at 0 -8 0)
 			(layer "F.SilkS")
@@
 		(descr "Kailh keyswitch Hotswap Socket plated holes Keycap 1.00u")
 		(tags "Kailh Keyboard Keyswitch Switch Hotswap Socket Plated Relief Cutout Keycap 1.00u")
-		(property "Reference" "SW5"
+		(property "Reference" "SW05"
 			(at 0 -8 0)
 			(layer "F.SilkS")
@@
 		(descr "Kailh keyswitch Hotswap Socket plated holes Keycap 1.00u")
 		(tags "Kailh Keyboard Keyswitch Switch Hotswap Socket Plated Relief Cutout Keycap 1.00u")
-		(property "Reference" "SW8"
+		(property "Reference" "SW08"
 			(at 0 -8 0)
 			(layer "F.SilkS")
@@
 		(descr "Kailh keyswitch Hotswap Socket plated holes Keycap 1.00u")
 		(tags "Kailh Keyboard Keyswitch Switch Hotswap Socket Plated Relief Cutout Keycap 1.00u")
-		(property "Reference" "SW4"
+		(property "Reference" "SW04"
 			(at 0 -8 0)
 			(layer "F.SilkS")
@@
 		(descr "Kailh keyswitch Hotswap Socket plated holes Keycap 1.00u")
 		(tags "Kailh Keyboard Keyswitch Switch Hotswap Socket Plated Relief Cutout Keycap 1.00u")
-		(property "Reference" "SW3"
+		(property "Reference" "SW03"
 			(at 0 -8 0)
 			(layer "F.SilkS")
