File: Original ErgonomicGamepad.kicad_sch (KiCad schematic)
At the start: 82 parts, among them J1 USB_C_Receptacle_USB2.0_16P, J2 Conn_01x08, J3 Conn_01x08, J4 Conn_01x08, J5 AVR-ISP-6, J6 Conn_01x08, J7 1824417, SW01 SW_DIP_x01, SW02 SW_DIP_x01, SW03 SW_DIP_x01, SW04 SW_DIP_x01, SW05 SW_DIP_x01, SW06 SW_DIP_x01, SW07 SW_DIP_x01, SW08 SW_DIP_x01, SW09 SW_DIP_x01, SW10 SW_DIP_x01, SW11 SW_DIP_x01, SW12 SW_DIP_x01, SW13 SW_DIP_x01, SW14 SW_DIP_x01, SW15 SW_DIP_x01, SW16 SW_DIP_x01, SW17 SW_DIP_x01, SW18 SW_DIP_x01, SW19 SW_DIP_x01, SW20 SW_DIP_x01, SW21 SW_DIP_x01, SW22 SW_DIP_x01, SW23 SW_DIP_x01, SW24 SW_DIP_x01, U1 ATmega32U4-A, U2 USBLC6-2SC6, Y1 Crystal

Commit message: chore: schematic runs ERC clean; parts need specification
Snapshot pin-remapping work plus JLC BOM tracking updates. Schematic
passes ERC with no errors, but most placed components still need
Manufacturer/MPN/Supplier/LCSC fields filled in (see
UnresolvedPartsPunchList.md for the full punch list).

Co-Authored-By: Claude Sonnet 5 <noreply@anthropic.com>
Parts:
- C1, C2, C3, C4, C5, D09, D10, D11, D12, D13, D15, D16, D17, D2, D20, D21, D22, D23, D24, D25, D26, D3, D4, D5, D6, D7, D8, D9, J2, J3, J4, J6, R1, R2, R3, R4, R5, R6, R7, SW01, SW02, SW03, SW04, SW05, SW06, SW07, SW08, SW09, SW10, SW11, SW12, SW13, SW14, SW15, SW16, SW17, SW18, SW19, SW20, SW21, SW22, SW23, SW24, SWR1, U1: Supplier LCSC -> (none)
- D1: LCSC C191023 -> (none); MPN 1N5819WS -> (none); Manufacturer Guangdong Hottech -> (none); Supplier LCSC -> (none)
- J1: LCSC C165948 -> (none); MPN TYPE-C-31-M-12 -> (none); Manufacturer Korean Hroparts Elec -> (none); Supplier LCSC -> (none)
- J5: footprint Connector_PinHeader_2.54mm:PinHeader_2x03_P2.54mm_Vertical_SMD -> Connector_PinHeader_2.54mm:PinHeader_2x03_P2.54mm_Vertical; LCSC C32713283 -> (none); MPN HX PZ2.54-2x3P TP -> (none); Manufacturer hanxia -> (none); Supplier LCSC -> (none)
- J7: value 1824417 -> Conn_01x02; footprint Connector_Phoenix_MC_HighVoltage:PhoenixContact_MCV_1,5_2-G-5.08_1x02_P5.08mm_Vertical -> Connector_PinHeader_2.54mm:PinHeader_1x02_P2.54mm_Vertical; LCSC C5873683 -> (none); MPN 1824417 -> (none); Manufacturer Phoenix Contact -> (none); Supplier LCSC -> (none)
- Y1: LCSC C13738 -> (none); MPN X322516MLB4SI -> (none); Manufacturer YXC Crystal Oscillators -> (none); Supplier LCSC -> (none)
