File: Was ErgonomicGamepad.kicad_sch (KiCad schematic)
At the start: 82 parts, among them J1 USB_C_Receptacle_USB2.0_16P, J2 Conn_01x08, J3 Conn_01x08, J4 Conn_01x08, J5 AVR-ISP-6, J6 Conn_01x08, J7 1824417, SW01 SW_DIP_x01, SW02 SW_DIP_x01, SW03 SW_DIP_x01, SW04 SW_DIP_x01, SW05 SW_DIP_x01, SW06 SW_DIP_x01, SW07 SW_DIP_x01, SW08 SW_DIP_x01, SW09 SW_DIP_x01, SW10 SW_DIP_x01, SW11 SW_DIP_x01, SW12 SW_DIP_x01, SW13 SW_DIP_x01, SW14 SW_DIP_x01, SW15 SW_DIP_x01, SW16 SW_DIP_x01, SW17 SW_DIP_x01, SW18 SW_DIP_x01, SW19 SW_DIP_x01, SW20 SW_DIP_x01, SW21 SW_DIP_x01, SW22 SW_DIP_x01, SW23 SW_DIP_x01, SW24 SW_DIP_x01, U1 ATmega32U4-A, U2 USBLC6-2SC6, Y1 Crystal

Commit message: chore: schematic runs ERC clean; parts need specification
Snapshot pin-remapping work plus JLC BOM tracking updates. Schematic
passes ERC with no errors, but most placed components still need
Manufacturer/MPN/Supplier/LCSC fields filled in (see
UnresolvedPartsPunchList.md for the full punch list).

Co-Authored-By: Claude Sonnet 5 <noreply@anthropic.com>
Parts:
- D1: LCSC C191023 -> (none); MPN 1N5819WS -> (none); Manufacturer Guangdong Hottech -> (none)
- J1: LCSC C165948 -> (none); MPN TYPE-C-31-M-12 -> (none); Manufacturer Korean Hroparts Elec -> (none)
- J5: footprint Connector_PinHeader_2.54mm:PinHeader_2x03_P2.54mm_Vertical_SMD -> Connector_PinHeader_2.54mm:PinHeader_2x03_P2.54mm_Vertical; LCSC C32713283 -> (none); MPN HX PZ2.54-2x3P TP -> (none); Manufacturer hanxia -> (none)
- J7: value 1824417 -> Conn_01x02; footprint Connector_Phoenix_MC_HighVoltage:PhoenixContact_MCV_1,5_2-G-5.08_1x02_P5.08mm_Vertical -> Connector_PinHeader_2.54mm:PinHeader_1x02_P2.54mm_Vertical; LCSC C5873683 -> (none); MPN 1824417 -> (none); Manufacturer Phoenix Contact -> (none)
- Y1: LCSC C13738 -> (none); MPN X322516MLB4SI -> (none); Manufacturer YXC Crystal Oscillators -> (none)
Changed lines of the file:
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@@
 			)
 		)
-		(property "Datasheet" "https://www.lcsc.com/datasheet/C13738.pdf"
+		(property "Datasheet" ""
 			(at 82.55 76.2 0)
 			(hide yes)
@@
 			)
 		)
-		(property "Manufacturer" "YXC Crystal Oscillators"
+		(property "Manufacturer" ""
 			(at 82.55 76.2 0)
 			(hide yes)
@@
 			)
 		)
-		(property "MPN" "X322516MLB4SI"
+		(property "MPN" ""
 			(at 82.55 76.2 0)
 			(hide yes)
@@
 			)
 		)
-		(property "LCSC" "C13738"
+		(property "LCSC" ""
 			(at 82.55 76.2 0)
 			(hide yes)
@@
 			)
 		)
-		(property "Datasheet" "https://www.lcsc.com/datasheet/C191023.pdf"
+		(property "Datasheet" "https://datasheet.lcsc.com/lcsc/2204281430_Guangdong-Hottech-1N5819WS_C191023.pdf"
 			(at 54.61 74.93 0)
 			(hide yes)
@@
 			)
 		)
-		(property "Manufacturer" "Guangdong Hottech"
+		(property "Manufacturer" ""
 			(at 54.61 74.93 90)
 			(hide yes)
@@
 			)
 		)
-		(property "MPN" "1N5819WS"
+		(property "MPN" ""
 			(at 54.61 74.93 90)
 			(hide yes)
@@
 			)
 		)
-		(property "LCSC" "C191023"
+		(property "LCSC" ""
 			(at 54.61 74.93 90)
 			(hide yes)
@@
 			)
 		)
-		(property "Footprint" "Connector_PinHeader_2.54mm:PinHeader_2x03_P2.54mm_Vertical_SMD"
+		(property "Footprint" "Connector_PinHeader_2.54mm:PinHeader_2x03_P2.54mm_Vertical"
 			(at 125.73 46.99 90)
 			(hide yes)
@@
 			)
 		)
-		(property "Datasheet" "https://www.lcsc.com/product-detail/C32713283.html"
+		(property "Datasheet" ""
 			(at 151.765 31.75 0)
 			(hide yes)
@@
 			)
 		)
-		(property "Manufacturer" "hanxia"
+		(property "Manufacturer" ""
 			(at 119.38 45.72 0)
 			(hide yes)
@@
 			)
 		)
-		(property "MPN" "HX PZ2.54-2x3P TP"
+		(property "MPN" ""
 			(at 119.38 45.72 0)
 			(hide yes)
@@
 			)
 		)
-		(property "LCSC" "C32713283"
+		(property "LCSC" ""
 			(at 119.38 45.72 0)
 			(hide yes)
@@
 			)
 		)
-		(property "Value" "1824417"
+		(property "Value" "Conn_01x02"
 			(at 29.21 40.6399 0)
 			(show_name no)
@@
 			)
 		)
-		(property "Footprint" "Connector_Phoenix_MC_HighVoltage:PhoenixContact_MCV_1,5_2-G-5.08_1x02_P5.08mm_Vertical"
+		(property "Footprint" "Connector_PinHeader_2.54mm:PinHeader_1x02_P2.54mm_Vertical"
 			(at 26.67 38.1 0)
 			(hide yes)
@@
 			)
 		)
-		(property "Datasheet" "https://www.lcsc.com/product-detail/C5873683.html"
+		(property "Datasheet" ""
 			(at 26.67 38.1 0)
 			(hide yes)
@@
 			)
 		)
-		(property "Description" "2-pin SMT power input connector"
+		(property "Description" "Generic connector, single row, 01x02, script generated (kicad-library-utils/schlib/autogen/connector/)"
 			(at 26.67 38.1 0)
 			(hide yes)
@@
 			)
 		)
-		(property "Manufacturer" "Phoenix Contact"
+		(property "Manufacturer" ""
 			(at 26.67 38.1 0)
 			(hide yes)
@@
 			)
 		)
-		(property "MPN" "1824417"
+		(property "MPN" ""
 			(at 26.67 38.1 0)
 			(hide yes)
@@
 			)
 		)
-		(property "LCSC" "C5873683"
+		(property "LCSC" ""
 			(at 26.67 38.1 0)
 			(hide yes)
@@
 			)
 		)
-		(property "Datasheet" "https://www.lcsc.com/datasheet/C165948.pdf"
+		(property "Datasheet" "https://www.usb.org/sites/default/files/documents/usb_type-c.zip"
 			(at 36.83 97.79 0)
 			(hide yes)
@@
 			)
 		)
-		(property "Manufacturer" "Korean Hroparts Elec"
+		(property "Manufacturer" ""
 			(at 33.02 97.79 0)
 			(hide yes)
@@
 			)
 		)
-		(property "MPN" "TYPE-C-31-M-12"
+		(property "MPN" ""
 			(at 33.02 97.79 0)
 			(hide yes)
@@
 			)
 		)
-		(property "LCSC" "C165948"
+		(property "LCSC" ""
 			(at 33.02 97.79 0)
 			(hide yes)
